Commit message: Use gz_ros2_control plugin & Gazebo Harmonic instead

File: ranger/ranger_mini/urdf/ranger_mini_gazebo.xacro (robot description, xacro)
@@ -13,4 +13,7 @@
                 <mesh filename="file://$(find ranger_mini)/meshes/ranger_base.dae" />
             </geometry>
+            <material name="dark_grey">
+                <color rgba="0.2 0.2 0.2 1.0"/>
+            </material>
         </visual>
         <collision>
@@ -335,7 +338,7 @@
       </actuator>
 	</transmission>
-  <ros2_control name="GazeboSystem" type="system">
+  <ros2_control name="GazeboSimSystem" type="system">
     <hardware>
-      <plugin>gazebo_ros2_control/GazeboSystem</plugin>
+      <plugin>gz_ros2_control/GazeboSimSystem</plugin>
     </hardware>
     <joint name="fl_wheel">
@@ -413,6 +416,8 @@
   </ros2_control>
     <gazebo>
-        <plugin name="gazebo_ros2_control" filename="libgazebo_ros2_control.so">
-            <parameters>/home/agilex/ugv_sim_ws/src/ugv_gazebo_sim/ranger/ranger_mini/config/ranger_mini_joint.yaml</parameters>
+        <plugin filename="libgz_ros2_control-system.so" name="gz_ros2_control::GazeboSimROS2ControlPlugin">
+            <robot_param>robot_description</robot_param>
+			<robot_param_node>robot_state_publisher</robot_param_node>
+            <parameters>/home/multirobots/multirobots_ws/src/ugv_gazebo_sim/ranger/ranger_mini/config/ranger_mini_joint.yaml</parameters>
         </plugin>
     </gazebo>

Commit message: Integration in the main simulation

File: ranger/ranger_mini/urdf/ranger_mini_gazebo.xacro (robot description, xacro)
@@ -1,4 +1,6 @@
 <?xml version="1.0"?>
 <robot name="ranger_mini_v2"  xmlns:xacro="http://ros.org/wiki/xacro">
+    <xacro:arg name="prefix" default="ranger_mini_"/>
+    <xacro:arg name="id" default="1"/>
     <!-- Base link -->
     <link name="base_link">
@@ -13,7 +15,7 @@
                 <mesh filename="file://$(find ranger_mini)/meshes/ranger_base.dae" />
             </geometry>
-            <material name="dark_grey">
+            <!-- <material name="dark_grey">
                 <color rgba="0.2 0.2 0.2 1.0"/>
-            </material>
+            </material> -->
         </visual>
         <collision>
@@ -170,35 +172,35 @@
         <limit effort="5" velocity="6.28"  lower="-2.1" upper="2.1" />
     </joint>
-        <link name="rl_wheel_link">
-            <inertial>
-                <mass value="8" />
-                <origin xyz="0 0 0" />
-                <inertia ixx="0.1171" ixy="0" ixz="0" iyy="0.1361" iyz="0" izz="0.1171" />
-            </inertial>
-            <visual>
-                <origin xyz="0 0 0" rpy="1.57 0 0" />
-                <geometry>
-                    <cylinder length="0.01" radius="0.01" />
-                </geometry>
-            </visual>
-            <collision>
-                <origin xyz="0 0 0" rpy="1.57 0 0" />
-                <geometry>
-                    <cylinder length="0.08" radius="0.08" />
-                </geometry>
-                     <contact>
-                         <ode>
-                        <min_depth>0.001</min_depth>
-                         </ode>
-                    </contact>
-            </collision>
-        </link>
-        <joint name="rl_wheel" type="continuous">
-            <origin xyz="0.0 0.0 -0.12 " rpy="0 0 0" />
-            <parent link="rl_steering_wheel_link"/>
-            <child link="rl_wheel_link"/>
-            <axis xyz="0 1 0" rpy="0 0 0" />
-            <limit effort="100" velocity="10" />
-        </joint>
+    <link name="rl_wheel_link">
+        <inertial>
+            <mass value="8" />
+            <origin xyz="0 0 0" />
+            <inertia ixx="0.1171" ixy="0" ixz="0" iyy="0.1361" iyz="0" izz="0.1171" />
+        </inertial>
+        <visual>
+            <origin xyz="0 0 0" rpy="1.57 0 0" />
+            <geometry>
+                <cylinder length="0.01" radius="0.01" />
+            </geometry>
+        </visual>
+        <collision>
+            <origin xyz="0 0 0" rpy="1.57 0 0" />
+            <geometry>
+                <cylinder length="0.08" radius="0.08" />
+            </geometry>
+                    <contact>
+                        <ode>
+                    <min_depth>0.001</min_depth>
+                        </ode>
+                </contact>
+        </collision>
+    </link>
+    <joint name="rl_wheel" type="continuous">
+        <origin xyz="0.0 0.0 -0.12 " rpy="0 0 0" />
+        <parent link="rl_steering_wheel_link"/>
+        <child link="rl_wheel_link"/>
+        <axis xyz="0 1 0" rpy="0 0 0" />
+        <limit effort="100" velocity="10" />
+    </joint>
    <link name="rr_steering_wheel_link">
         <inertial>
@@ -227,35 +229,35 @@
         <limit effort="5" velocity="6.28"  lower="-2.1" upper="2.1" />
     </joint>
-        <link name="rr_wheel_link">
-            <inertial>
-                <mass value="8" />
-                <origin xyz="0 0 0" />
-                <inertia ixx="0.1171" ixy="0" ixz="0" iyy="0.1361" iyz="0" izz="0.1171" />
-            </inertial>
-            <visual>
-                <origin xyz="0.0 0.0 0.0" rpy="1.57 0 0" />
-                <geometry>
-                    <cylinder length="0.01" radius="0.01" />
-                </geometry>
-            </visual>
-            <collision>
-                <origin xyz="0 0 0" rpy="1.57 0 0" />
-                <geometry>
-                    <cylinder length="0.08" radius="0.08" />
-                </geometry>
-                     <contact>
-                         <ode>
-                        <min_depth>0.001</min_depth>
-                         </ode>
-                    </contact>
-            </collision>
-        </link>
-        <joint name="rr_wheel" type="continuous">
-            <origin xyz="0.0 0.0 -0.12 " rpy="0 0 0" />
-            <parent link="rr_steering_wheel_link"/>
-            <child link="rr_wheel_link"/>
-            <axis xyz="0 1 0" rpy="0 0 0" />
-            <limit effort="100" velocity="10" />
-        </joint>
+    <link name="rr_wheel_link">
+        <inertial>
+            <mass value="8" />
+            <origin xyz="0 0 0" />
+            <inertia ixx="0.1171" ixy="0" ixz="0" iyy="0.1361" iyz="0" izz="0.1171" />
+        </inertial>
+        <visual>
+            <origin xyz="0.0 0.0 0.0" rpy="1.57 0 0" />
+            <geometry>
+                <cylinder length="0.01" radius="0.01" />
+            </geometry>
+        </visual>
+        <collision>
+            <origin xyz="0 0 0" rpy="1.57 0 0" />
+            <geometry>
+                <cylinder length="0.08" radius="0.08" />
+            </geometry>
+                    <contact>
+                        <ode>
+                    <min_depth>0.001</min_depth>
+                        </ode>
+                </contact>
+        </collision>
+    </link>
+    <joint name="rr_wheel" type="continuous">
+        <origin xyz="0.0 0.0 -0.12 " rpy="0 0 0" />
+        <parent link="rr_steering_wheel_link"/>
+        <child link="rr_wheel_link"/>
+        <axis xyz="0 1 0" rpy="0 0 0" />
+        <limit effort="100" velocity="10" />
+    </joint>
 	<transmission name="fl_steering_wheel_trans">
       <type>transmission_interface/SimpleTransmission</type>
@@ -338,87 +340,136 @@
       </actuator>
 	</transmission>
-  <ros2_control name="GazeboSimSystem" type="system">
-    <hardware>
-      <plugin>gz_ros2_control/GazeboSimSystem</plugin>
-    </hardware>
-    <joint name="fl_wheel">
-      <command_interface name="velocity">
-        <param name="min">-3.14</param>
-        <param name="max">3.14</param>
-      </command_interface>
-      <state_interface name="velocity"/>
-      <state_interface name="effort"/>
-      <state_interface name="position"/>
-    </joint>
-    <joint name="fr_wheel">
-      <command_interface name="velocity">
-        <param name="min">-3.14</param>
-        <param name="max">3.14</param>
-      </command_interface>
-      <state_interface name="velocity"/>
-      <state_interface name="effort"/>
-      <state_interface name="position"/>
-    </joint>
-    <joint name="rl_wheel">
-      <command_interface name="velocity">
-        <param name="min">-3.14</param>
-        <param name="max">3.14</param>
-      </command_interface>
-      <state_interface name="velocity"/>
-      <state_interface name="effort"/>
-      <state_interface name="position"/>
-    </joint>
-    <joint name="rr_wheel">
-      <command_interface name="velocity">
-        <param name="min">-3.14</param>
-        <param name="max">3.14</param>
-      </command_interface>
-      <state_interface name="velocity"/>
-      <state_interface name="effort"/>
-      <state_interface name="position"/>
-    </joint>
-    <joint name="fl_steering_wheel">
-      <command_interface name="position">
-        <param name="min">-3.14</param>
-        <param name="max">3.14</param>
-      </command_interface>
-      <state_interface name="position"/>
-      <state_interface name="velocity"/>
-      <state_interface name="effort"/>
-    </joint>
-    <joint name="fr_steering_wheel">
-      <command_interface name="position">
-        <param name="min">-3.14</param>
-        <param name="max">3.14</param>
-      </command_interface>
-      <state_interface name="position"/>
-      <state_interface name="velocity"/>
-      <state_interface name="effort"/>
-    </joint>
-    <joint name="rl_steering_wheel">
-      <command_interface name="position">
-        <param name="min">-3.14</param>
-        <param name="max">3.14</param>
-      </command_interface>
-      <state_interface name="position"/>
-      <state_interface name="velocity"/>
-      <state_interface name="effort"/>
-    </joint>
-    <joint name="rr_steering_wheel">
-      <command_interface name="position">
-        <param name="min">-3.14</param>
-        <param name="max">3.14</param>
-      </command_interface>
-      <state_interface name="position"/>
-      <state_interface name="velocity"/>
-      <state_interface name="effort"/>
-    </joint>
-  </ros2_control>
-    <gazebo>
-        <plugin filename="libgz_ros2_control-system.so" name="gz_ros2_control::GazeboSimROS2ControlPlugin">
-            <robot_param>robot_description</robot_param>
-			<robot_param_node>robot_state_publisher</robot_param_node>
-            <parameters>/home/multirobots/multirobots_ws/src/ugv_gazebo_sim/ranger/ranger_mini/config/ranger_mini_joint.yaml</parameters>
-        </plugin>
-    </gazebo>
+    <xacro:include filename="$(find robotnik_sensors)/urdf/all_sensors.urdf.xacro" />
+    <xacro:macro name="sensors" params="id prefix">
+        <!-- IMU -->
+		<xacro:sensor_pixhawk id="$(arg id)" frame_prefix="$(arg prefix)imu_" name_prefix="$(arg prefix)" parent="base_link">
+			<origin xyz="-0.12 0.0 0.01" rpy="0 0 0"/>
+		</xacro:sensor_pixhawk>
+		<!-- 2d lidar -->
+		<xacro:sensor_hokuyo_urg04lx id="$(arg id)" frame_prefix="$(arg prefix)front_laser_" name_prefix="$(arg prefix)" parent="base_link">
+			<origin xyz="0.0 0.0 0.0" rpy="0 0 0"/>
+		</xacro:sensor_hokuyo_urg04lx>
+		<!-- GPS -->
+	  	<xacro:sensor_gps id="$(arg id)" frame_prefix="$(arg prefix)gps_" name_prefix="$(arg prefix)" parent="base_link">
+			<origin xyz="-0.22 0 0.0" rpy="0 0 0"/>
+		</xacro:sensor_gps>
+		<!-- ptz camera -->
+		<!-- <xacro:sensor_axis_m5013 id="$(arg id)" frame_prefix="$(arg prefix)camera_" name_prefix="$(arg prefix)" parent="base_link">
+			<origin xyz="0.185 0 0.23" rpy="0 ${-75*PI/180} 0"/>
+		</xacro:sensor_axis_m5013> -->
+		<!-- depth camera -->
+		<xacro:sensor_azure_kinect id="$(arg id)" frame_prefix="$(arg prefix)depth_camera_" name_prefix="$(arg prefix)" parent="base_link">
+			<!-- <origin xyz="0.324 0.012 0.172" rpy="0 0 ${PI/2}"/> -->
+			<origin xyz="0.41 0.06 -0.08" rpy="0 0 ${PI/2}"/>
+		</xacro:sensor_azure_kinect>
+    </xacro:macro>
+    <xacro:sensors id="$(arg id)" prefix="$(arg prefix)"/>
+    <xacro:macro name="ros_control" params="id prefix">
+        <ros2_control name="GazeboSimSystem" type="system">
+            <hardware>
+                <plugin>gz_ros2_control/GazeboSimSystem</plugin>
+            </hardware>
+            <joint name="fl_wheel">
+                <command_interface name="velocity">
+                    <param name="min">-3.14</param>
+                    <param name="max">3.14</param>
+                </command_interface>
+                <state_interface name="velocity"/>
+                <state_interface name="effort"/>
+                <state_interface name="position"/>
+            </joint>
+            <joint name="fr_wheel">
+                <command_interface name="velocity">
+                    <param name="min">-3.14</param>
+                    <param name="max">3.14</param>
+                </command_interface>
+                <state_interface name="velocity"/>
+                <state_interface name="effort"/>
+                <state_interface name="position"/>
+            </joint>
+            <joint name="rl_wheel">
+                <command_interface name="velocity">
+                    <param name="min">-3.14</param>
+                    <param name="max">3.14</param>
+                </command_interface>
+                <state_interface name="velocity"/>
+                <state_interface name="effort"/>
+                <state_interface name="position"/>
+            </joint>
+            <joint name="rr_wheel">
+                <command_interface name="velocity">
+                    <param name="min">-3.14</param>
+                    <param name="max">3.14</param>
+                </command_interface>
+                <state_interface name="velocity"/>
+                <state_interface name="effort"/>
+                <state_interface name="position"/>
+            </joint>
+            <joint name="fl_steering_wheel">
+                <command_interface name="position">
+                    <param name="min">-3.14</param>
+                    <param name="max">3.14</param>
+                </command_interface>
+                <state_interface name="position"/>
+                <state_interface name="velocity"/>
+                <state_interface name="effort"/>
+            </joint>
+            <joint name="fr_steering_wheel">
+                <command_interface name="position">
+                    <param name="min">-3.14</param>
+                    <param name="max">3.14</param>
+                </command_interface>
+                <state_interface name="position"/>
+                <state_interface name="velocity"/>
+                <state_interface name="effort"/>
+            </joint>
+            <joint name="rl_steering_wheel">
+                <command_interface name="position">
+                    <param name="min">-3.14</param>
+                    <param name="max">3.14</param>
+                </command_interface>
+                <state_interface name="position"/>
+                <state_interface name="velocity"/>
+                <state_interface name="effort"/>
+            </joint>
+            <joint name="rr_steering_wheel">
+                <command_interface name="position">
+                    <param name="min">-3.14</param>
+                    <param name="max">3.14</param>
+                </command_interface>
+                <state_interface name="position"/>
+                <state_interface name="velocity"/>
+                <state_interface name="effort"/>
+            </joint>
+            <joint name="ranger_mini_camera_pan_joint">
+				<command_interface name="position">
+					<param name="min">-3.1416</param>
+					<param name="max">3.1416</param>
+				</command_interface>
+				<state_interface name="position"/>
+				<state_interface name="velocity"/>
+				<state_interface name="effort"/>
+			</joint>
+			<joint name="ranger_mini_camera_tilt_joint">
+				<command_interface name="position">
+					<param name="min">-1.5708</param>
+					<param name="max">1.5708</param>
+				</command_interface>
+				<state_interface name="position"/>
+				<state_interface name="velocity"/>
+				<state_interface name="effort"/>
+			</joint>
+        </ros2_control>
+        <gazebo>
+            <plugin filename="libgz_ros2_control-system.so" name="gz_ros2_control::GazeboSimROS2ControlPlugin">
+                <robot_param>robot_description</robot_param>
+                <robot_param_node>robot_state_publisher</robot_param_node>
+                <parameters>/tmp/${prefix}${id}_control.yaml</parameters>
+                <ros>
+                    <namespace>${prefix}${id}</namespace>
+                </ros>
+            </plugin>
+        </gazebo>
+    </xacro:macro>
+    <xacro:ros_control id="$(arg id)" prefix="$(arg prefix)"/>
 </robot>
